Commit message: Experimenting with buoyancy.

File: src/snake_control/urdf/rotary_module.xacro (robot description, xacro)
@@ -2,5 +2,5 @@
 <robot xmlns:xacro="http://www.ros.org/wiki/xacro">
   <xacro:property name="PI" value="3.1415926535897931" />
-  <xacro:property name="mass_2" value="1.35" />
+  <xacro:property name="mass_2" value="1.575" />
   <xacro:property name="cyl_r" value="0.0335" />
   <xacro:property name="cyl_h_in" value="0.03" />

File: src/snake_control/urdf/snake.xacro (robot description, xacro)
@@ -16,5 +16,5 @@
     <parent link="kdl_dummy_root"/>
     <child link="base"/>
-    <origin xyz="0 0 0" rpy="0 ${-PI/2.0} 0"/>
+    <origin xyz="0 0 0" rpy="${-PI/2.0} 0 0"/>
   </joint>
   <link name="base" />
