Commit message: Gaits: revised and reworked.

File: src/snake_control/urdf/module_common.xacro (robot description, xacro)
@@ -2,4 +2,26 @@
 <robot xmlns:xacro="http://www.ros.org/wiki/xacro">
   <xacro:property name="PI" value="3.1415926535897931" />
+  <!-- define macros for colors: -->
+  <xacro:macro name="red_material">
+    <material name="red">
+      <color rgba=".82 0.06 0.06 1"/>
+    </material>
+  </xacro:macro>
+  <xacro:macro name="silver_material">
+    <material name="silver">
+      <color rgba="0.6 0.6 0.6 1"/>
+    </material>
+  </xacro:macro>
+  <xacro:macro name="black_material">
+    <material name="black">
+      <color rgba="0 0 0 1"/>
+    </material>
+  </xacro:macro>
+  <xacro:macro name="fluorescent_material">
+    <material name="fluorescent">
+      <color rgba="0.8 1 0 1"/>
+    </material>
+  </xacro:macro>
+  <!-- define collar element macro -->
   <xacro:macro name="collar" params="parent">
     <link name="${parent}__COLLAR">
@@ -9,4 +31,5 @@
           <mesh filename="package://snake_control/meshes/collar.dae"/>
         </geometry>
+        <xacro:black_material/>
       </visual>
     </link>
@@ -16,19 +39,18 @@
     </joint>
   </xacro:macro>
-  <xacro:macro name="just_collar" params="name">
-    <link name="${name}">
+  <xacro:macro name="end" params="parent">
+    <link name="${parent}__COLLAR_END">
       <visual>
-        <origin xyz="0 0.0004965 -0.0065" rpy="${PI/2.0} ${PI} ${PI}" />
+        <origin xyz="0 0.0004965 +0.03" rpy="${PI/2.0} ${PI} ${PI}" />
         <geometry>
           <mesh filename="package://snake_control/meshes/collar.dae"/>
         </geometry>
+        <xacro:black_material/>
       </visual>
-      <collision>
-        <origin xyz="0 0 -0.0065" rpy="0 0 0" />
-        <geometry>
-        <cylinder radius="${0.0335}" length="${0.0175}" />
-        </geometry>
-      </collision>
     </link>
+    <joint name="${parent}__COLLAR_JOINT" type="fixed">
+      <parent link="${parent}"/>
+      <child link="${parent}__COLLAR_END"/>
+    </joint>
   </xacro:macro>
 </robot>

File: src/snake_control/urdf/rotary_module.xacro (robot description, xacro)
@@ -2,9 +2,8 @@
 <robot xmlns:xacro="http://www.ros.org/wiki/xacro">
   <xacro:property name="PI" value="3.1415926535897931" />
-  <xacro:property name="mass_2" value="1.575" />
+  <xacro:property name="mass_2" value="0.093195" />
   <xacro:property name="cyl_r" value="0.0335" />
   <xacro:property name="cyl_h_in" value="0.03" />
   <xacro:property name="cyl_h_out" value="0.03" />
-  <xacro:property name="cyl_h_end" value="0.0765" />
   <xacro:macro name="rotary_module_in" params="name">
     <link name="${name}">
@@ -14,4 +13,5 @@
           <mesh filename="package://snake_control/meshes/rotary_module_in.dae"/>
         </geometry>
+        <xacro:red_material/>
       </visual>
     <collision>
@@ -54,10 +54,12 @@
         <geometry>
           <mesh filename="package://snake_control/meshes/rotary_module_out.dae"/>
+	  <!-- <cylinder radius=".0025" length=".1" /> -->
         </geometry>
+        <xacro:red_material/>
       </visual>
     <collision>
       <origin xyz="0 0 0" rpy="0 0 0" />
       <geometry>
-	    <cylinder radius="${cyl_r}" length="${cyl_h_out}" />
+	<cylinder radius="${cyl_r}" length="${cyl_h_out}" />
       </geometry>
     </collision>
@@ -76,12 +78,15 @@
     </joint>
   </xacro:macro>
+  <!-- NOTE: joint must match the name of the module -->
   <xacro:macro name="rotary_module" params="joint child">
-    <!-- fixed joint + collar -->
+    <!-- first half of joint + collar -->
     <xacro:rotary_module_in name="${joint}__INPUT_INTERFACE"/>
     <xacro:collar parent="${joint}__INPUT_INTERFACE"/>
-    <!-- rotary joint -->
-    <xacro:rotary_module_joint parent="${joint}__INPUT_INTERFACE" name="${joint}_joint" child="${joint}"/>
-    <xacro:rotary_module_out name="${joint}"/>
-    <xacro:rotary_module_out_interface parent="${joint}" name="${joint}__OUTPUT_INTERFACE" child="${child}__INPUT_INTERFACE"/>
+    <!-- actual rotary joint component: -->
+    <xacro:rotary_module_joint parent="${joint}__INPUT_INTERFACE" name="${joint}" child="${joint}__OUTPUT_BODY"/>
+    <!-- second half of joint -->
+    <xacro:rotary_module_out name="${joint}__OUTPUT_BODY"/>
+    <!-- 90* turn at interface: -->
+    <xacro:rotary_module_out_interface parent="${joint}__OUTPUT_BODY" name="${joint}__OUTPUT_INTERFACE" child="${child}__INPUT_INTERFACE"/>
   </xacro:macro>
 </robot>

File: src/snake_control/urdf/snake.xacro (robot description, xacro)
@@ -1,20 +1,23 @@
 <?xml version="1.0"?>
 <robot xmlns:xacro="http://www.ros.org/wiki/xacro" name="snake">
+  <!-- *************************** XACRO MACROS *************************** -->
   <xacro:property name="PI" value="3.1415926535897931" />
+  <!-- load macros for modules -->
   <xacro:include filename="./module_common.xacro"/>
   <xacro:include filename="./rotary_module.xacro"/>
-  <!-- ************************* Arboc definition ************************* -->
-  <xacro:property name="S_00" value="link_1" />
-  <xacro:property name="S_01" value="link_2" />
-  <xacro:property name="S_02" value="link_3" />
-  <xacro:property name="S_03" value="link_4" />
-  <xacro:property name="S_04" value="link_5" />
-  <xacro:property name="S_05" value="link_6" />
-  <xacro:property name="S_06" value="link_7" />
-  <link name="kdl_dummy_root" />
-  <joint name="kdl_dummy_root_to_base" type="fixed">
-    <parent link="kdl_dummy_root"/>
+  <!-- ************************* ROBOT DEFINITION ************************* -->
+  <xacro:property name="S_00" value="link_01" />
+  <xacro:property name="S_01" value="link_02" />
+  <xacro:property name="S_02" value="link_03" />
+  <xacro:property name="S_03" value="link_04" />
+  <xacro:property name="S_04" value="link_05" />
+  <xacro:property name="S_05" value="link_06" />
+  <xacro:property name="S_06" value="link_07" />
+  <xacro:property name="S_07" value="link_08" />
+  <link name="dummy_root" />
+  <joint name="dummy_root_to_base" type="fixed">
+    <parent link="dummy_root"/>
     <child link="base"/>
-    <origin xyz="0 0 0" rpy="${-PI/2.0} 0 0"/>
+    <origin xyz="0 0 0" rpy="0 0 0"/>
   </joint>
   <link name="base" />
@@ -30,4 +33,10 @@
   <xacro:rotary_module joint="${S_04}" child="${S_05}"/>
   <xacro:rotary_module joint="${S_05}" child="${S_06}"/>
-  <xacro:just_collar name="${S_06}__INPUT_INTERFACE"/>
+  <xacro:rotary_module joint="${S_06}" child="${S_07}"/>
+  <xacro:rotary_module_in name="${S_07}__INPUT_INTERFACE"/>
+  <xacro:collar parent="${S_07}__INPUT_INTERFACE"/>
+  <xacro:rotary_module_joint parent="${S_07}__INPUT_INTERFACE" name="${S_07}" child="${S_07}__OUTPUT_BODY"/>
+  <xacro:rotary_module_out name="${S_07}__OUTPUT_BODY"/>
+  <xacro:end parent="${S_07}__OUTPUT_BODY"/>
+  <!-- ********************** Arboc attempt ********************** -->
 </robot>
